File: hardware/interface.sch (EAGLE design)
At the start: 17 parts, among them J1 DCJ0202

Commit message: cleaned up the interface.sch
Connections:
- net N$8 renamed RPI_PIN16
- removed net N$6: C5.1, GPIO_PIN_ON_BOARD.18, R3.1
- removed net N$7: U$6.COIL1, ULN2003.10
- removed net OUT: C4.1, LM3940.OUT, R2.1
- removed net VCC: U$6.COIL2, U$6.MAIN, ULN2003.8
- new net +3V3: C4.1, LM3940.OUT, R2.1, U$6.COIL1, ULN2003.8
- new net +5V: C2.1, C3.1, LM3940.IN, LM7805.OUT, R1.2, U$6.MAIN
- new net RPI_PIN17: C5.1, GPIO_PIN_ON_BOARD.17, R3.1
- net N$2: now also U$6.COIL2, ULN2003.10; no longer C2.1, C3.1, LM3940.IN, LM7805.OUT, R1.2
Other:
- note added: "Interfacing circuit for Alarm"
- note added: "Interfacing circuit for Door Sensor/switch"
- note added: "Power Supply Section"
- note removed: "+3V3"
- note removed: "+5V0"
- note removed: "Operating Volt to Relay"
- moved on the sheet: BELL, C1, C2, C3, C4, C5, GPIO_PIN_ON_BOARD, J1, LM3940, LM7805, R1, R2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
